File: power-bus/hardware/power-bus.sch (KiCad schematic (older format))
At the start: 18 parts, among them J1 CONN_01X02, J10 CONN_01X02, J11 CONN_01X02, J12 CONN_01X02, J13 CONN_01X02, J2 CONN_01X02, J3 CONN_01X02, J4 CONN_01X02, J5 CONN_01X02, J6 CONN_01X02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

Commit message: Mounting holes, logos.
Parts:
- added M1, M2, M3: MOUNT_HOLE, conservify:HOLE_NPTH_3.2MM, symbol MOUNT_HOLE
- added M4: MOUNT_HOLE, RocketScreamKicadLibrary:HOLE_PTH_3.2MM, symbol MOUNT_HOLE
Changed lines of the file:
@@
 Wire Wire Line
 	2650 4900 2400 4900
+$Comp
+L MOUNT_HOLE M1
+U 1 1 59023B33
+P 5050 2600
+F 0 "M1" H 5050 2750 50  0000 C CNN
+F 1 "MOUNT_HOLE" H 5050 2450 50  0001 C CNN
+F 2 "conservify:HOLE_NPTH_3.2MM" H 5075 2375 50  0001 C CNN
+F 3 "" H 5050 2600 50  0000 C CNN
+	1    5050 2600
+	1    0    0    -1
+$EndComp
+$Comp
+L MOUNT_HOLE M2
+U 1 1 59023BD7
+P 5250 2600
+F 0 "M2" H 5250 2750 50  0000 C CNN
+F 1 "MOUNT_HOLE" H 5250 2450 50  0001 C CNN
+F 2 "conservify:HOLE_NPTH_3.2MM" H 5275 2375 50  0001 C CNN
+F 3 "" H 5250 2600 50  0000 C CNN
+	1    5250 2600
+	1    0    0    -1
+$EndComp
+$Comp
+L MOUNT_HOLE M3
+U 1 1 59023C27
+P 5450 2600
+F 0 "M3" H 5450 2750 50  0000 C CNN
+F 1 "MOUNT_HOLE" H 5450 2450 50  0001 C CNN
+F 2 "conservify:HOLE_NPTH_3.2MM" H 5475 2375 50  0001 C CNN
+F 3 "" H 5450 2600 50  0000 C CNN
+	1    5450 2600
+	1    0    0    -1
+$EndComp
+$Comp
+L MOUNT_HOLE M4
+U 1 1 59023C7E
+P 5650 2600
+F 0 "M4" H 5650 2750 50  0000 C CNN
+F 1 "MOUNT_HOLE" H 5650 2450 50  0001 C CNN
+F 2 "RocketScreamKicadLibrary:HOLE_PTH_3.2MM" H 5675 2375 50  0001 C CNN
+F 3 "" H 5650 2600 50  0000 C CNN
+	1    5650 2600
+	1    0    0    -1
+$EndComp
 $EndSCHEMATC

Commit message: Add better mounting holes, some labels, etc...
Parts:
- removed J12: CONN_01X02, Connectors_Terminal_Blocks:TerminalBlock_Pheonix_MKDS1.5-2pol, symbol CONN_01X02
- removed J13: CONN_01X02, Socket_Strips:Socket_Strip_Straight_1x02_Pitch2.54mm, symbol CONN_01X02
- added J8: CONN_01X02, Connectors_Terminal_Blocks:TerminalBlock_Pheonix_MKDS1.5-2pol, symbol CONN_01X02
- M1, M2, M3: footprint conservify:HOLE_NPTH_3.2MM -> conservify:HOLE_NPTH_3.8MM
- M4: footprint RocketScreamKicadLibrary:HOLE_PTH_3.2MM -> conservify:HOLE_NPTH_3.8MM
Connections:
- wire segments 50 -> 48
Other:
- moved on the sheet: J1
Changed lines of the file:
@@
 L CONN_01X02 J1
 U 1 1 58FA5FA2
-P 800 950
-F 0 "J1" H 800 1100 50  0000 C CNN
-F 1 "CONN_01X02" V 900 950 50  0000 C CNN
-F 2 "Connectors_Terminal_Blocks:TerminalBlock_Pheonix_MKDS1.5-2pol" H 800 950 50  0001 C CNN
-F 3 "" H 800 950 50  0001 C CNN
-	1    800  950
+P 800 850
+F 0 "J1" H 800 1000 50  0000 C CNN
+F 1 "CONN_01X02" V 900 850 50  0000 C CNN
+F 2 "Connectors_Terminal_Blocks:TerminalBlock_Pheonix_MKDS1.5-2pol" H 800 850 50  0001 C CNN
+F 3 "" H 800 850 50  0001 C CNN
+	1    800  850
 	-1   0    0    1
 $EndComp
@@
 Text Label 1950 900  0    60   ~ 0
 VRAW
-Text Label 1300 1000 0    60   ~ 0
+Text Label 1300 800  0    60   ~ 0
 GND
 Text Label 3050 1500 0    60   ~ 0
@@
 	1600 900  1000 900
 Wire Wire Line
-	1600 1000 1000 1000
+	1600 800  1000 800
 Wire Wire Line
 	3050 1400 3550 1400
@@
 	6550 1700 6200 1700
 $Comp
-L GND #PWR01
+L GND #PWR1
 U 1 1 58FA74B4
-P 2300 950
-F 0 "#PWR01" H 2300 700 50  0001 C CNN
-F 1 "GND" H 2300 800 50  0000 C CNN
-F 2 "" H 2300 950 50  0001 C CNN
-F 3 "" H 2300 950 50  0001 C CNN
-	1    2300 950
-	1    0    0    -1
-$EndComp
-Text Label 2450 900  0    60   ~ 0
-GND
-Wire Wire Line
-	2700 900  2300 900
-Wire Wire Line
-	2300 900  2300 950
+P 1050 1800
+F 0 "#PWR1" H 1050 1550 50  0001 C CNN
+F 1 "GND" H 1050 1650 50  0000 C CNN
+F 2 "" H 1050 1800 50  0001 C CNN
+F 3 "" H 1050 1800 50  0001 C CNN
+	1    1050 1800
+	1    0    0    -1
+$EndComp
+Text Label 1200 1750 0    60   ~ 0
+GND
+Wire Wire Line
+	1450 1750 1050 1750
+Wire Wire Line
+	1050 1750 1050 1800
 $Comp
 L CONN_01X02 J10
@@
 Wire Wire Line
 	1950 3850 1600 3850
-$Comp
-L CONN_01X02 J12
-U 1 1 58FA881A
-P 5100 1650
-F 0 "J12" H 5100 1800 50  0000 C CNN
-F 1 "CONN_01X02" V 5200 1650 50  0000 C CNN
-F 2 "Connectors_Terminal_Blocks:TerminalBlock_Pheonix_MKDS1.5-2pol" H 5100 1650 50  0001 C CNN
-F 3 "" H 5100 1650 50  0001 C CNN
-	1    5100 1650
-	-1   0    0    1
-$EndComp
-Text Label 5350 1700 0    60   ~ 0
-VADJ_1
-Text Label 5350 1600 0    60   ~ 0
-GND
-Wire Wire Line
-	5650 1600 5300 1600
-Wire Wire Line
-	5650 1700 5300 1700
 $Comp
 L pololu-vreg U2
@@
 VIN
 $Comp
-L CONN_01X02 J13
-U 1 1 58FE47A9
-P 2850 4850
-F 0 "J13" H 2850 5000 50  0000 C CNN
-F 1 "CONN_01X02" V 2950 4850 50  0000 C CNN
-F 2 "Socket_Strips:Socket_Strip_Straight_1x02_Pitch2.54mm" H 2850 4850 50  0001 C CNN
-F 3 "" H 2850 4850 50  0001 C CNN
-	1    2850 4850
-	1    0    0    -1
-$EndComp
-Text Label 2400 4800 0    60   ~ 0
-GND
-Text Label 2400 4900 0    60   ~ 0
-GND
-Wire Wire Line
-	2400 4800 2650 4800
-Wire Wire Line
-	2650 4900 2400 4900
-$Comp
 L MOUNT_HOLE M1
 U 1 1 59023B33
@@
 F 0 "M1" H 5050 2750 50  0000 C CNN
 F 1 "MOUNT_HOLE" H 5050 2450 50  0001 C CNN
-F 2 "conservify:HOLE_NPTH_3.2MM" H 5075 2375 50  0001 C CNN
+F 2 "conservify:HOLE_NPTH_3.8MM" H 5075 2375 50  0001 C CNN
 F 3 "" H 5050 2600 50  0000 C CNN
 	1    5050 2600
@@
 F 0 "M2" H 5250 2750 50  0000 C CNN
 F 1 "MOUNT_HOLE" H 5250 2450 50  0001 C CNN
-F 2 "conservify:HOLE_NPTH_3.2MM" H 5275 2375 50  0001 C CNN
+F 2 "conservify:HOLE_NPTH_3.8MM" H 5275 2375 50  0001 C CNN
 F 3 "" H 5250 2600 50  0000 C CNN
 	1    5250 2600
@@
 F 0 "M3" H 5450 2750 50  0000 C CNN
 F 1 "MOUNT_HOLE" H 5450 2450 50  0001 C CNN
-F 2 "conservify:HOLE_NPTH_3.2MM" H 5475 2375 50  0001 C CNN
+F 2 "conservify:HOLE_NPTH_3.8MM" H 5475 2375 50  0001 C CNN
 F 3 "" H 5450 2600 50  0000 C CNN
 	1    5450 2600
@@
 F 0 "M4" H 5650 2750 50  0000 C CNN
 F 1 "MOUNT_HOLE" H 5650 2450 50  0001 C CNN
-F 2 "RocketScreamKicadLibrary:HOLE_PTH_3.2MM" H 5675 2375 50  0001 C CNN
+F 2 "conservify:HOLE_NPTH_3.8MM" H 5675 2375 50  0001 C CNN
 F 3 "" H 5650 2600 50  0000 C CNN
 	1    5650 2600
 	1    0    0    -1
 $EndComp
+$Comp
+L CONN_01X02 J8
+U 1 1 59024BCB
+P 800 1500
+F 0 "J8" H 800 1650 50  0000 C CNN
+F 1 "CONN_01X02" V 900 1500 50  0000 C CNN
+F 2 "Connectors_Terminal_Blocks:TerminalBlock_Pheonix_MKDS1.5-2pol" H 800 1500 50  0001 C CNN
+F 3 "" H 800 1500 50  0001 C CNN
+	1    800  1500
+	-1   0    0    1
+$EndComp
+Text Label 1150 1450 0    60   ~ 0
+VRAW
+Text Label 1150 1550 0    60   ~ 0
+GND
+Wire Wire Line
+	1450 1450 1000 1450
+Wire Wire Line
+	1450 1550 1000 1550
 $EndSCHEMATC

Commit message: Fix fuse footprint.
Parts:
- F1: footprint Fuse_Holders_and_Fuses:Fuseholder5x20_horiz_open_universal_Type-III -> conservify:Fuseholder6x30_horiz_open_inline_Type-I
Changed lines of the file:
@@
 	6550 1700 6200 1700
 $Comp
-L GND #PWR1
+L GND #PWR01
 U 1 1 58FA74B4
 P 1050 1800
-F 0 "#PWR1" H 1050 1550 50  0001 C CNN
+F 0 "#PWR01" H 1050 1550 50  0001 C CNN
 F 1 "GND" H 1050 1650 50  0000 C CNN
 F 2 "" H 1050 1800 50  0001 C CNN
@@
 F 0 "F1" V 1830 900 50  0000 C CNN
 F 1 "Fuse" V 1675 900 50  0000 C CNN
-F 2 "Fuse_Holders_and_Fuses:Fuseholder5x20_horiz_open_universal_Type-III" V 1680 900 50  0001 C CNN
+F 2 "conservify:Fuseholder6x30_horiz_open_inline_Type-I" V 1680 900 50  0001 C CNN
 F 3 "" H 1750 900 50  0001 C CNN
 	1    1750 900
