File: power-bus/power-bus.sch (KiCad schematic (older format))
At the start: 21 parts, among them J1 CONN_01X02, J10 CONN_01X02, J11 CONN_01X02, J2 CONN_01X02, J3 CONN_01X02, J4 CONN_01X02, J5 CONN_01X02, J6 CONN_01X02, J7 CONN_01X02, J8 CONN_01X02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

Commit message: Add more Vraw connectors to the power bus board.
Parts:
- removed J3, J7: CONN_01X02, Connectors_Terminal_Blocks:TerminalBlock_Pheonix_MKDS1.5-2pol, symbol CONN_01X02
- removed U2, U5: pololu-vreg, conservify:pololu-vreg-adjustable, symbol pololu-vreg
- added J12, J13: CONN_01X02, conservify:TerminalBlock_Phoenix_MKDS1.5-2pol, symbol CONN_01X02
- J1, J10, J11, J2, J4, J5, J6, J8: footprint Connectors_Terminal_Blocks:TerminalBlock_Pheonix_MKDS1.5-2pol -> conservify:TerminalBlock_Phoenix_MKDS1.5-2pol
Connections:
- net labels removed: 12V0_3, 12V0_3_EN
- wire segments 48 -> 39
Other:
- moved on the sheet: J8
Changed lines of the file:
@@
 F 0 "J1" H 800 1000 50  0000 C CNN
 F 1 "CONN_01X02" V 900 850 50  0000 C CNN
-F 2 "Connectors_Terminal_Blocks:TerminalBlock_Pheonix_MKDS1.5-2pol" H 800 850 50  0001 C CNN
+F 2 "conservify:TerminalBlock_Phoenix_MKDS1.5-2pol" H 800 850 50  0001 C CNN
 F 3 "" H 800 850 50  0001 C CNN
 	1    800  850
@@
 F 0 "J2" H 2300 1800 50  0000 C CNN
 F 1 "CONN_01X02" V 2400 1650 50  0000 C CNN
-F 2 "Connectors_Terminal_Blocks:TerminalBlock_Pheonix_MKDS1.5-2pol" H 2300 1650 50  0001 C CNN
+F 2 "conservify:TerminalBlock_Phoenix_MKDS1.5-2pol" H 2300 1650 50  0001 C CNN
 F 3 "" H 2300 1650 50  0001 C CNN
 	1    2300 1650
@@
 Text Label 2550 1600 0    60   ~ 0
 GND
-$Comp
-L pololu-vreg U3
-U 1 1 58FA64F5
-P 4300 3100
-F 0 "U3" H 4300 3200 60  0000 C CNN
-F 1 "pololu-vreg" H 4300 3100 60  0000 C CNN
-F 2 "conservify:pololu-vreg-adjustable" H 4300 3100 60  0001 C CNN
-F 3 "" H 4300 3100 60  0001 C CNN
-	1    4300 3100
-	1    0    0    -1
-$EndComp
-Text Label 3050 3050 0    60   ~ 0
-VRAW
-Text Label 3050 3150 0    60   ~ 0
-GND
-Text Label 3050 3250 0    60   ~ 0
-12V0_1
-Text Label 3050 2950 0    60   ~ 0
-12V0_1_EN
 $Comp
 L pololu-vreg U4
@@
 12V0_2_EN
 $Comp
-L CONN_01X02 J4
-U 1 1 58FA6511
-P 2300 3200
-F 0 "J4" H 2300 3350 50  0000 C CNN
-F 1 "CONN_01X02" V 2400 3200 50  0000 C CNN
-F 2 "Connectors_Terminal_Blocks:TerminalBlock_Pheonix_MKDS1.5-2pol" H 2300 3200 50  0001 C CNN
-F 3 "" H 2300 3200 50  0001 C CNN
-	1    2300 3200
-	-1   0    0    1
-$EndComp
-$Comp
 L CONN_01X02 J5
 U 1 1 58FA6517
@@
 F 0 "J5" H 2300 4050 50  0000 C CNN
 F 1 "CONN_01X02" V 2400 3900 50  0000 C CNN
-F 2 "Connectors_Terminal_Blocks:TerminalBlock_Pheonix_MKDS1.5-2pol" H 2300 3900 50  0001 C CNN
+F 2 "conservify:TerminalBlock_Phoenix_MKDS1.5-2pol" H 2300 3900 50  0001 C CNN
 F 3 "" H 2300 3900 50  0001 C CNN
 	1    2300 3900
@@
 Text Label 2550 3950 0    60   ~ 0
 12V0_2
-Text Label 2550 3250 0    60   ~ 0
-12V0_1
-Text Label 2550 3150 0    60   ~ 0
-GND
-$Comp
-L pololu-vreg U5
-U 1 1 58FA671E
-P 8000 1550
-F 0 "U5" H 8000 1650 60  0000 C CNN
-F 1 "pololu-vreg" H 8000 1550 60  0000 C CNN
-F 2 "conservify:pololu-vreg-adjustable" H 8000 1550 60  0001 C CNN
-F 3 "" H 8000 1550 60  0001 C CNN
-	1    8000 1550
-	1    0    0    -1
-$EndComp
-Text Label 6750 1500 0    60   ~ 0
-VRAW
-Text Label 6750 1600 0    60   ~ 0
-GND
-Text Label 6750 1700 0    60   ~ 0
-VADJ_1
-Text Label 6750 1400 0    60   ~ 0
-VADJ_1_EN
 $Comp
 L CONN_01X02 J6
@@
 F 0 "J6" H 6000 1800 50  0000 C CNN
 F 1 "CONN_01X02" V 6100 1650 50  0000 C CNN
-F 2 "Connectors_Terminal_Blocks:TerminalBlock_Pheonix_MKDS1.5-2pol" H 6000 1650 50  0001 C CNN
+F 2 "conservify:TerminalBlock_Phoenix_MKDS1.5-2pol" H 6000 1650 50  0001 C CNN
 F 3 "" H 6000 1650 50  0001 C CNN
 	1    6000 1650
@@
 	2850 1700 2500 1700
 Wire Wire Line
-	3050 2950 3550 2950
-Wire Wire Line
-	3050 3050 3550 3050
-Wire Wire Line
-	3050 3150 3550 3150
-Wire Wire Line
-	3050 3250 3550 3250
-Wire Wire Line
 	3050 3650 3550 3650
 Wire Wire Line
@@
 Wire Wire Line
 	2850 3850 2500 3850
-Wire Wire Line
-	2850 3150 2500 3150
-Wire Wire Line
-	2850 3250 2500 3250
-Wire Wire Line
-	6750 1400 7250 1400
-Wire Wire Line
-	6750 1500 7250 1500
-Wire Wire Line
-	6750 1600 7250 1600
-Wire Wire Line
-	6750 1700 7250 1700
 Wire Wire Line
 	6550 1600 6200 1600
@@
 	1050 1750 1050 1800
 $Comp
-L CONN_01X02 J10
-U 1 1 58FA8646
-P 1400 3200
-F 0 "J10" H 1400 3350 50  0000 C CNN
-F 1 "CONN_01X02" V 1500 3200 50  0000 C CNN
-F 2 "Connectors_Terminal_Blocks:TerminalBlock_Pheonix_MKDS1.5-2pol" H 1400 3200 50  0001 C CNN
-F 3 "" H 1400 3200 50  0001 C CNN
-	1    1400 3200
-	-1   0    0    1
-$EndComp
-Text Label 1650 3250 0    60   ~ 0
-12V0_1
-Text Label 1650 3150 0    60   ~ 0
-GND
-Wire Wire Line
-	1950 3150 1600 3150
-Wire Wire Line
-	1950 3250 1600 3250
-$Comp
 L CONN_01X02 J11
 U 1 1 58FA8689
@@
 F 0 "J11" H 1400 4050 50  0000 C CNN
 F 1 "CONN_01X02" V 1500 3900 50  0000 C CNN
-F 2 "Connectors_Terminal_Blocks:TerminalBlock_Pheonix_MKDS1.5-2pol" H 1400 3900 50  0001 C CNN
+F 2 "conservify:TerminalBlock_Phoenix_MKDS1.5-2pol" H 1400 3900 50  0001 C CNN
 F 3 "" H 1400 3900 50  0001 C CNN
 	1    1400 3900
@@
 Wire Wire Line
 	1950 3850 1600 3850
-$Comp
-L pololu-vreg U2
-U 1 1 58FE353A
-P 4300 2400
-F 0 "U2" H 4300 2500 60  0000 C CNN
-F 1 "pololu-vreg" H 4300 2400 60  0000 C CNN
-F 2 "conservify:pololu-vreg-adjustable" H 4300 2400 60  0001 C CNN
-F 3 "" H 4300 2400 60  0001 C CNN
-	1    4300 2400
-	1    0    0    -1
-$EndComp
-Text Label 3050 2350 0    60   ~ 0
-VRAW
-Text Label 3050 2450 0    60   ~ 0
-GND
-Text Label 3050 2550 0    60   ~ 0
-12V0_3
-Text Label 3050 2250 0    60   ~ 0
-12V0_3_EN
-$Comp
-L CONN_01X02 J7
-U 1 1 58FE3544
-P 2300 2500
-F 0 "J7" H 2300 2650 50  0000 C CNN
-F 1 "CONN_01X02" V 2400 2500 50  0000 C CNN
-F 2 "Connectors_Terminal_Blocks:TerminalBlock_Pheonix_MKDS1.5-2pol" H 2300 2500 50  0001 C CNN
-F 3 "" H 2300 2500 50  0001 C CNN
-	1    2300 2500
-	-1   0    0    1
-$EndComp
-Text Label 2550 2450 0    60   ~ 0
-GND
-Text Label 2550 2550 0    60   ~ 0
-12V0_3
-Wire Wire Line
-	3050 2250 3550 2250
-Wire Wire Line
-	3050 2350 3550 2350
-Wire Wire Line
-	3050 2450 3550 2450
-Wire Wire Line
-	3050 2550 3550 2550
-Wire Wire Line
-	2850 2550 2500 2550
-Wire Wire Line
-	2850 2450 2500 2450
-$Comp
-L CONN_01X02 J3
-U 1 1 58FE3552
-P 1400 2500
-F 0 "J3" H 1400 2650 50  0000 C CNN
-F 1 "CONN_01X02" V 1500 2500 50  0000 C CNN
-F 2 "Connectors_Terminal_Blocks:TerminalBlock_Pheonix_MKDS1.5-2pol" H 1400 2500 50  0001 C CNN
-F 3 "" H 1400 2500 50  0001 C CNN
-	1    1400 2500
-	-1   0    0    1
-$EndComp
-Text Label 1650 2450 0    60   ~ 0
-GND
-Text Label 1650 2550 0    60   ~ 0
-12V0_3
-Wire Wire Line
-	1950 2550 1600 2550
-Wire Wire Line
-	1950 2450 1600 2450
 $Comp
 L CONN_01X05 J9
@@
 	1    0    0    -1
 $EndComp
-Text Label 3800 4550 0    60   ~ 0
-12V0_3_EN
-Text Label 3800 4650 0    60   ~ 0
-12V0_1_EN
 Text Label 3800 4750 0    60   ~ 0
 12V0_2_EN
@@
 Text Label 3800 4950 0    60   ~ 0
 GND
-Wire Wire Line
-	3800 4550 4350 4550
 Wire Wire Line
 	3800 4650 4350 4650
@@
 L CONN_01X02 J8
 U 1 1 59024BCB
-P 800 1500
-F 0 "J8" H 800 1650 50  0000 C CNN
-F 1 "CONN_01X02" V 900 1500 50  0000 C CNN
-F 2 "Connectors_Terminal_Blocks:TerminalBlock_Pheonix_MKDS1.5-2pol" H 800 1500 50  0001 C CNN
-F 3 "" H 800 1500 50  0001 C CNN
-	1    800  1500
-	-1   0    0    1
-$EndComp
-Text Label 1150 1450 0    60   ~ 0
-VRAW
-Text Label 1150 1550 0    60   ~ 0
-GND
-Wire Wire Line
-	1450 1450 1000 1450
-Wire Wire Line
-	1450 1550 1000 1550
+P 1400 5000
+F 0 "J8" H 1400 5150 50  0000 C CNN
+F 1 "CONN_01X02" V 1500 5000 50  0000 C CNN
+F 2 "conservify:TerminalBlock_Phoenix_MKDS1.5-2pol" H 1400 5000 50  0001 C CNN
+F 3 "" H 1400 5000 50  0001 C CNN
+	1    1400 5000
+	-1   0    0    1
+$EndComp
+Text Label 1750 4950 0    60   ~ 0
+VRAW
+Text Label 1750 5050 0    60   ~ 0
+GND
+Wire Wire Line
+	2050 4950 1600 4950
+Wire Wire Line
+	2050 5050 1600 5050
+$Comp
+L CONN_01X02 J12
+U 1 1 5A0A3125
+P 1400 4500
+F 0 "J12" H 1400 4650 50  0000 C CNN
+F 1 "CONN_01X02" V 1500 4500 50  0000 C CNN
+F 2 "conservify:TerminalBlock_Phoenix_MKDS1.5-2pol" H 1400 4500 50  0001 C CNN
+F 3 "" H 1400 4500 50  0001 C CNN
+	1    1400 4500
+	-1   0    0    1
+$EndComp
+Text Label 1750 4450 0    60   ~ 0
+VRAW
+Text Label 1750 4550 0    60   ~ 0
+GND
+Wire Wire Line
+	2050 4450 1600 4450
+Wire Wire Line
+	2050 4550 1600 4550
+$Comp
+L CONN_01X02 J13
+U 1 1 5A0A35B3
+P 1400 5500
+F 0 "J13" H 1400 5650 50  0000 C CNN
+F 1 "CONN_01X02" V 1500 5500 50  0000 C CNN
+F 2 "conservify:TerminalBlock_Phoenix_MKDS1.5-2pol" H 1400 5500 50  0001 C CNN
+F 3 "" H 1400 5500 50  0001 C CNN
+	1    1400 5500
+	-1   0    0    1
+$EndComp
+Text Label 1750 5450 0    60   ~ 0
+VRAW
+Text Label 1750 5550 0    60   ~ 0
+GND
+Wire Wire Line
+	2050 5450 1600 5450
+Wire Wire Line
+	2050 5550 1600 5550
+Text Label 3050 2950 0    60   ~ 0
+12V0_1_EN
+Wire Wire Line
+	3050 2950 3550 2950
+Wire Wire Line
+	1950 3250 1600 3250
+Wire Wire Line
+	1950 3150 1600 3150
+Text Label 1650 3150 0    60   ~ 0
+GND
+Text Label 1650 3250 0    60   ~ 0
+12V0_1
+$Comp
+L CONN_01X02 J10
+U 1 1 58FA8646
+P 1400 3200
+F 0 "J10" H 1400 3350 50  0000 C CNN
+F 1 "CONN_01X02" V 1500 3200 50  0000 C CNN
+F 2 "conservify:TerminalBlock_Phoenix_MKDS1.5-2pol" H 1400 3200 50  0001 C CNN
+F 3 "" H 1400 3200 50  0001 C CNN
+	1    1400 3200
+	-1   0    0    1
+$EndComp
+Wire Wire Line
+	2850 3250 2500 3250
+Wire Wire Line
+	2850 3150 2500 3150
+Wire Wire Line
+	3050 3250 3550 3250
+Wire Wire Line
+	3050 3150 3550 3150
+Wire Wire Line
+	3050 3050 3550 3050
+Text Label 2550 3150 0    60   ~ 0
+GND
+Text Label 2550 3250 0    60   ~ 0
+12V0_1
+$Comp
+L CONN_01X02 J4
+U 1 1 58FA6511
+P 2300 3200
+F 0 "J4" H 2300 3350 50  0000 C CNN
+F 1 "CONN_01X02" V 2400 3200 50  0000 C CNN
+F 2 "conservify:TerminalBlock_Phoenix_MKDS1.5-2pol" H 2300 3200 50  0001 C CNN
+F 3 "" H 2300 3200 50  0001 C CNN
+	1    2300 3200
+	-1   0    0    1
+$EndComp
+Text Label 3050 3250 0    60   ~ 0
+12V0_1
+Text Label 3050 3150 0    60   ~ 0
+GND
+Text Label 3050 3050 0    60   ~ 0
+VRAW
+$Comp
+L pololu-vreg U3
+U 1 1 58FA64F5
+P 4300 3100
+F 0 "U3" H 4300 3200 60  0000 C CNN
+F 1 "pololu-vreg" H 4300 3100 60  0000 C CNN
+F 2 "conservify:pololu-vreg-adjustable" H 4300 3100 60  0001 C CNN
+F 3 "" H 4300 3100 60  0001 C CNN
+	1    4300 3100
+	1    0    0    -1
+$EndComp
+Text Label 3800 4650 0    60   ~ 0
+12V0_1_EN
 $EndSCHEMATC
